File: PCB/EasyTalkie.kicad_pcb (KiCad board)
At the start: 2 copper layers, 55.2 x 81.8 mm, 6 parts, among them SW1 SW_Push, SW2 ON/OFF, U1 XIAO-ESP32-S3-DIP, U2 INMP441, U3 MAX98357A

Commit message: cad
Other:
- board size 55.2 x 81.8 mm -> 55 x 82 mm
Changed lines of the file:
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@@
 		(layer "F.SilkS")
 	)
-	(gr_rect
-		(start 188 23.5)
-		(end 243.25 105.25)
+	(gr_arc
+		(start 190.5 105.5)
+		(mid 188.732233 104.767767)
+		(end 188 103)
 		(stroke
 			(width 0.05)
 			(type default)
 		)
-		(fill no)
 		(layer "Edge.Cuts")
 	)
+	(gr_line
+		(start 240.5 105.5)
+		(end 190.5 105.5)
+		(stroke
+			(width 0.05)
+			(type default)
+		)
+		(layer "Edge.Cuts")
+	)
+	(gr_line
+		(start 190.5 23.5)
+		(end 240.5 23.5)
+		(stroke
+			(width 0.05)
+			(type default)
+		)
+		(layer "Edge.Cuts")
+	)
+	(gr_line
+		(start 188 103)
+		(end 188 26)
+		(stroke
+			(width 0.05)
+			(type default)
+		)
+		(layer "Edge.Cuts")
+	)
+	(gr_arc
+		(start 243 103)
+		(mid 242.267767 104.767767)
+		(end 240.5 105.5)
+		(stroke
+			(width 0.05)
+			(type default)
+		)
+		(layer "Edge.Cuts")
+	)
+	(gr_arc
+		(start 240.5 23.5)
+		(mid 242.267767 24.232233)
+		(end 243 26)
+		(stroke
+			(width 0.05)
+			(type default)
+		)
+		(layer "Edge.Cuts")
+	)
+	(gr_arc
+		(start 188 26)
+		(mid 188.732233 24.232233)
+		(end 190.5 23.5)
+		(stroke
+			(width 0.05)
+			(type default)
+		)
+		(layer "Edge.Cuts")
+	)
+	(gr_line
+		(start 243 26)
+		(end 243 103)
+		(stroke
+			(width 0.05)
+			(type default)
+		)
+		(layer "Edge.Cuts")
+	)

Commit message: fix
Parts:
- SW2: value ON/OFF -> ~
- U4: value ~ -> SSD1306
Connections:
- net GPI07 renamed GPI043
Other:
- board text added: "AMP HERE"
- board text added: "EASYTALKIE"
- board text added: "ESP32 S3 Here"
- board text added: "INMP441"
- board text added: "OFF/ON"
Changed lines of the file:
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@@
 	(net 5 "GPI04")
 	(net 6 "Net-(U3-OUTP)")
-	(net 7 "GPI07")
+	(net 7 "GPI043")
 	(net 8 "Net-(U3-OUTN)")
 	(net 9 "GPI05")
@@
 		)
 		(property "Value" "INMP441"
-			(at 5.7 0 0)
+			(at 0 8.44 0)
 			(layer "F.Fab")
 			(effects
@@
 			)
 		)
-		(property "Value" "~"
+		(property "Value" "SSD1306"
 			(at -7.747 -7.62 0)
 			(layer "F.Fab")
@@
 			)
 		)
-		(property "Value" "ON/OFF"
+		(property "Value" "~"
 			(at 0.00762 -2.75082 90)
 			(layer "F.SilkS")
@@
 			(layers "*.Cu" "*.Mask")
 			(remove_unused_layers no)
-			(net 7 "GPI07")
+			(net 7 "GPI043")
 			(pinfunction "GPIO43_D6_TX")
 			(pintype "passive")
@@
 			(layers "B.Cu" "B.Mask")
 			(roundrect_rratio 0.1)
-			(net 7 "GPI07")
+			(net 7 "GPI043")
 			(pinfunction "GPIO43_D6_TX")
 			(pintype "passive")
@@
 			(layers "*.Cu" "*.Mask")
 			(remove_unused_layers no)
-			(net 7 "GPI07")
+			(net 7 "GPI043")
 			(pinfunction "DIN")
 			(pintype "input")
@@
 		)
 	)
+	(gr_text "EASYTALKIE"
+		(at 189.25 104 0)
+		(layer "F.SilkS")
+		(effects
+			(font
+				(size 1.5 1.5)
+				(thickness 0.375)
+				(bold yes)
+			)
+			(justify left bottom)
+		)
+	)
+	(gr_text "INMP441"
+		(at 197.75 78.75 0)
+		(layer "F.SilkS")
+		(effects
+			(font
+				(size 1 1)
+				(thickness 0.1)
+			)
+			(justify left bottom)
+		)
+	)
+	(gr_text "OFF/ON"
+		(at 195 97.75 90)
+		(layer "F.SilkS")
+		(effects
+			(font
+				(size 1 1)
+				(thickness 0.1)
+			)
+			(justify left bottom)
+		)
+	)
+	(gr_text "ESP32 S3 Here"
+		(at 204.25 38.5 -0)
+		(layer "B.SilkS")
+		(effects
+			(font
+				(size 1 1)
+				(thickness 0.1)
+			)
+			(justify left bottom mirror)
+		)
+	)
+	(gr_text "AMP HERE"
+		(at 234.5 43.25 270)
+		(layer "B.SilkS")
+		(effects
+			(font
+				(size 1 1)
+				(thickness 0.1)
+			)
+			(justify left bottom mirror)
+		)
+	)

Commit message: fix
Connections:
- SW2 pad 2: BAT+ -> LIPO BATTERY+
- SW2 pad 3: LIPO BATTERY+ -> BAT+
Changed lines of the file:
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@@
 			(layers "*.Cu" "*.Mask" "F.SilkS")
 			(remove_unused_layers no)
-			(net 19 "BAT+")
+			(net 17 "LIPO BATTERY+")
 			(pinfunction "COM")
 			(pintype "input")
@@
 			(layers "*.Cu" "*.Mask" "F.SilkS")
 			(remove_unused_layers no)
-			(net 17 "LIPO BATTERY+")
+			(net 19 "BAT+")
 			(pinfunction "B")
 			(pintype "input")
