File: PCB/EasyTalkie.kicad_sch (KiCad schematic)
At the start: 8 parts, among them J1 Battery, SW1 SW_Push, U1 XIAO-ESP32-S3-DIP, U2 INMP441, U3 MAX98357A

Commit message: pcb
Parts:
- U4: value ~ -> SSD1306
Other:
- moved on the sheet: J1, LS1, SW1, SW2, U1, U2, U3, U4

Commit message: firmware
Connections:
- net GPI07 renamed GPI043
Changed lines of the file:
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@@
 		)
 	)
-	(global_label "GPI07"
+	(global_label "GPI043"
 		(shape input)
 		(at 50.8 54.61 180)
@@
 		)
 		(property "Intersheetrefs" "${INTERSHEET_REFS}"
-			(at 42.251 54.61 0)
+			(at 41.0415 54.61 0)
 			(effects
 				(font
@@
 		)
 	)
-	(global_label "GPI07"
+	(global_label "GPI043"
 		(shape input)
 		(at 35.56 162.56 180)
@@
 		)
 		(property "Intersheetrefs" "${INTERSHEET_REFS}"
-			(at 27.011 162.56 0)
+			(at 25.8015 162.56 0)
 			(effects
 				(font

Commit message: fix
Connections:
- net BAT- is gone; now on net BAT+: U1. (BAT-)
- net BAT+: now also SW2.3 (B); no longer SW2.2 (COM)
- net LIPO BATTERY+: now also SW2.2 (COM); no longer SW2.3 (B)
